Commit message: fix: integrate Astra diagonal mounting pair

File: urdf/lekiwi_cad.urdf (robot description, URDF)
Before this commit: robot LeKiwi, 36 links, 35 joints
Joints:
- joint astra_pro_compact_mount_joint: origin xyz=-0.1 0 0.007 rpy=0 0 1.5707963267948966 -> xyz=-0.09 -0.04 0.007 rpy=0 0 2.0344439357957027

Commit message: build: add complete robot model rebuild

File: urdf/lekiwi_cad.urdf (robot description, URDF)
Before this commit: robot LeKiwi, 36 links, 35 joints
Joints:
- joint astra_pro_compact_mount_joint: origin xyz=-0.09 -0.04 0.007 rpy=0 0 2.0344439357957027 -> xyz=-0.09 -0.04 0.007 rpy=0.0 0.0 2.0344439357957027
- joint robotskin_lidar_mount_joint: origin xyz=0.0 -0.115 0.007 rpy=0 0 -1.5707963267948966 -> xyz=0.0 -0.115 0.007 rpy=0.0 0.0 -1.5707963267948966

Commit message: fix: stabilize model and simulation qualification

File: urdf/lekiwi_cad.urdf (robot description, URDF)
Before this commit: robot LeKiwi, 36 links, 35 joints
Joints:
- joint 94868A713_NO-THREADS_Female-Threaded-Hex-Standoff_Rigid-21: origin xyz=0.0 0.0 -0.05 rpy=3.141592653589793 -0.0 0.0 -> xyz=0.06 0.08 -0.05 rpy=3.141592653589793 -0.0 0.0
- joint base_plate_layer1-v5_Rigid-20: origin xyz=0.0 0.0 0.0 rpy=3.141592653589793 -0.0 0.0 -> xyz=-0.06 0.08 0 rpy=3.141592653589793 -0.0 0.0
- joint base_plate_layer1-v5_Rigid-30: origin xyz=0.02 -0.1 0.0 rpy=3.141592653589793 -0.0 0.0 -> xyz=0.06 -0.08 0 rpy=3.141592653589793 -0.0 0.0
- joint base_plate_layer1-v5_Rigid-31: origin xyz=0.07660254 0.06732051 0.0 rpy=3.141592653589793 -0.0 0.0 -> xyz=0.06 0.08 0 rpy=3.141592653589793 -0.0 0.0
- joint base_plate_layer1-v5_Rigid-32: origin xyz=-0.09660254 0.032679490000000005 0.0 rpy=3.141592653589793 -0.0 0.0 -> xyz=-0.06 -0.08 0 rpy=3.141592653589793 -0.0 0.0
- joint base_plate_layer1-v5_Rigid-69: origin xyz=0.1 -0.02 0.0 rpy=3.141592653589793 -0.0 0.0 -> xyz=0.1 0 0 rpy=3.141592653589793 -0.0 0.0
- joint base_plate_layer1-v5_Rigid-70: origin xyz=-0.1 -0.02 0.0 rpy=3.141592653589793 -0.0 0.0 -> xyz=-0.1 0 0 rpy=3.141592653589793 -0.0 0.0
- joint base_plate_layer1-v5_baseplate2bottom_mount: origin xyz=-0.02 -0.1 0.0 rpy=3.141592653589793 -0.0 0.0 -> xyz=0.02375 -0.06895 0 rpy=1.57079632679 0 -1.57079632679
- joint base_plate_layer1-v5_baseplate2left_mount: origin xyz=-0.05928203 0.057320510000000005 0.0 rpy=3.141592653589793 -0.0 0.0 -> xyz=-0.0715874515909 0.0139068966601 0 rpy=1.57079632679 2.77555756156e-17 2.61799387799
- joint base_plate_layer1-v5_baseplate2right_mount: origin xyz=0.07928203 0.022679490000000004 0.0 rpy=0.0 -0.0 0.0 -> xyz=0.0478374515909 0.0550431033399 0 rpy=1.57079632679 0 0.523598775598
- joint drive_motor_mount-v11-1_Rigid-35: origin xyz=-0.007786400000000002 -0.018513550000000004 0.0076100000000000004 rpy=-7.401486830834375e-17 -1.5707963267948966 0 -> xyz=0.00555000203031 0.0429865595601 0.0339999998126 rpy=-3.66519142919 1.57079632679 0
- joint drive_motor_mount-v11-2_Rigid-2: origin xyz=-0.01214 -0.015999999999999997 -0.0076100000000000004 rpy=3.141592653589793 1.5707963267948966 0 -> xyz=0.00555000019073 0.0429865544308 0.0339999998126 rpy=-1.57079632679 1.57079632679 0
- joint drive_motor_mount-v11_Rigid-39: origin xyz=0.019926399999999997 -0.0025135499999999933 -0.0076100000000000004 rpy=3.141592653589793 1.5707963267948966 0 -> xyz=0.00555000555268 0.0429865554023 0.0339999998126 rpy=-5.75958653158 1.57079632679 0

Commit message: fix: align shoulder limit with valid robot pose

File: urdf/lekiwi_cad.urdf (robot description, URDF)
Before this commit: robot LeKiwi, 39 links, 38 joints
Joints:
- joint arm_shoulder_lift: limit lower=-1.74533 upper=1.74533 effort=4 velocity=2 -> lower=-1.74533 upper=1.82 effort=4 velocity=2
