Commit message: feat: harden cleanroom robot qualification

File: urdf/lekiwi.urdf.xacro (robot description, xacro)
@@ -3,8 +3,11 @@
 <robot xmlns:xacro="http://www.ros.org/wiki/xacro" name="lekiwi">
   <xacro:arg name="sim" default="false"/>
-  <!-- Gazebo has no arm actuator in this stack. Keep its arm rigid in sim,
-       matching the previous model, while the real description stays movable. -->
-  <xacro:property name="arm_joint" value="${'fixed' if '$(arg sim)'.lower() == 'true' else 'revolute'}"/>
-  <xacro:property name="roll_joint" value="${'fixed' if '$(arg sim)'.lower() == 'true' else 'continuous'}"/>
+  <!-- The simulator now drives the same six bounded joints as the hardware.
+       Keep the joint type identical in both descriptions so a plan validated
+       in Gazebo has the same kinematic constraints on the physical robot. -->
+  <xacro:property name="arm_joint" value="revolute"/>
+  <!-- The physical wrist cable and servo have a bounded safe travel envelope.
+       Declaring it continuous makes MoveIt discard the configured bounds. -->
+  <xacro:property name="roll_joint" value="revolute"/>
   <!-- Vendored from robotmindio/LeKiwi at efa608d; see urdf/README.md. -->
   <xacro:include filename="lekiwi_cad.urdf"/>
@@ -99,14 +102,84 @@
     <origin xyz="0 0 0.220" rpy="0 0 0"/>
   </joint>
-  <!-- Preserve the original Gazebo mobile-base, lidar, and front-camera
-       functionality. References use the normalized ROS wrapper frames. -->
+  <!-- Gazebo-only contact and actuator model.  The CAD wheel meshes and their
+       measured mass remain vendored and untouched.  These small invisible
+       spheres supply the roller contact that the visual-only CAD lacks.  Each
+       axle is radial; positive rotation therefore drives tangentially in the
+       same [240, 0, 120]-90 degree convention as LeRobot's kinematics. -->
   <xacro:if value="$(arg sim)">
+    <xacro:macro name="sim_omni_wheel" params="name xyz axis">
+      <link name="${name}_contact">
+        <inertial>
+          <mass value="0.005"/>
+          <inertia ixx="0.000005" ixy="0" ixz="0" iyy="0.000005" iyz="0" izz="0.000005"/>
+        </inertial>
+        <collision name="contact">
+          <geometry><sphere radius="0.050"/></geometry>
+        </collision>
+      </link>
+      <joint name="${name}_joint" type="continuous">
+        <parent link="base_link"/><child link="${name}_contact"/>
+        <origin xyz="${xyz}" rpy="0 0 0"/>
+        <axis xyz="${axis}"/>
+        <dynamics damping="0.02" friction="0.01"/>
+        <limit effort="1.2" velocity="12.0"/>
+      </joint>
+      <gazebo>
+        <plugin filename="gz-sim-joint-controller-system" name="gz::sim::systems::JointController">
+          <joint_name>${name}_joint</joint_name>
+          <!-- The model-local watchdog is the only writer to the native
+               controller.  The public topic remains bridge-compatible. -->
+          <topic>/sim/${name}/native_cmd_vel</topic>
+          <!-- The ROS-side controller ramps every target with measured
+               acceleration and jerk limits. Gazebo then constrains that wheel
+               rate through contact; applying another PID here produced a
+               drivetrain-dependent hidden ramp and asymmetric tracking. -->
+        </plugin>
+      </gazebo>
+    </xacro:macro>
+    <!-- Wheel centres use the 0.125 m radius assumed by the hardware firmware.
+         z=-0.043 puts the 50 mm contact radius on z=0 when base_link is 93 mm
+         above base_footprint. -->
+    <xacro:sim_omni_wheel name="sim_base_left_wheel" xyz="0.0625 0.108253 -0.043" axis="-0.5 -0.866025 0"/>
+    <xacro:sim_omni_wheel name="sim_base_back_wheel" xyz="-0.125 0 -0.043" axis="1 0 0"/>
+    <xacro:sim_omni_wheel name="sim_base_right_wheel" xyz="0.0625 -0.108253 -0.043" axis="-0.5 0.866025 0"/>
     <gazebo>
-      <plugin filename="gz-sim-velocity-control-system" name="gz::sim::systems::VelocityControl">
-        <topic>/cmd_vel</topic>
+      <!-- Gazebo-native fail-safe: public bridge topics are forwarded only
+           while fresh. If ros_gz_bridge or either ROS adapter disappears,
+           it actively zeros wheel demand and interrupts the native arm
+           trajectory with a current-position hold. -->
+      <plugin filename="liblekiwi_sim_native_failsafe.so" name="lekiwi_rmf::SimNativeFailsafe"/>
+      <plugin filename="gz-sim-joint-state-publisher-system" name="gz::sim::systems::JointStatePublisher">
+        <topic>/sim/joint_states</topic><update_rate>50</update_rate>
+        <joint_name>sim_base_left_wheel_joint</joint_name>
+        <joint_name>sim_base_back_wheel_joint</joint_name>
+        <joint_name>sim_base_right_wheel_joint</joint_name>
+        <joint_name>arm_shoulder_pan</joint_name>
+        <joint_name>arm_shoulder_lift</joint_name>
+        <joint_name>arm_elbow_flex</joint_name>
+        <joint_name>arm_wrist_flex</joint_name>
+        <joint_name>arm_wrist_roll</joint_name>
+        <joint_name>arm_gripper</joint_name>
       </plugin>
-      <plugin filename="gz-sim-odometry-publisher-system" name="gz::sim::systems::OdometryPublisher">
-        <odom_frame>odom</odom_frame><robot_base_frame>base_footprint</robot_base_frame>
-        <odom_topic>/odom</odom_topic><tf_topic>/tf</tf_topic><dimensions>2</dimensions>
+      <plugin filename="gz-sim-joint-trajectory-controller-system" name="gz::sim::systems::JointTrajectoryController">
+        <topic>/sim/arm/native_joint_trajectory</topic>
+        <joint_name>arm_shoulder_pan</joint_name><initial_position>0</initial_position>
+        <position_p_gain>18</position_p_gain><position_i_gain>0.2</position_i_gain><position_d_gain>0.8</position_d_gain>
+        <position_cmd_min>-4</position_cmd_min><position_cmd_max>4</position_cmd_max>
+        <joint_name>arm_shoulder_lift</joint_name><initial_position>0</initial_position>
+        <position_p_gain>70</position_p_gain><position_i_gain>0.3</position_i_gain><position_d_gain>2.0</position_d_gain>
+        <position_cmd_min>-4</position_cmd_min><position_cmd_max>4</position_cmd_max>
+        <joint_name>arm_elbow_flex</joint_name><initial_position>0</initial_position>
+        <position_p_gain>70</position_p_gain><position_i_gain>0.3</position_i_gain><position_d_gain>2.0</position_d_gain>
+        <position_cmd_min>-4</position_cmd_min><position_cmd_max>4</position_cmd_max>
+        <joint_name>arm_wrist_flex</joint_name><initial_position>0</initial_position>
+        <position_p_gain>12</position_p_gain><position_i_gain>0.1</position_i_gain><position_d_gain>0.4</position_d_gain>
+        <position_cmd_min>-2</position_cmd_min><position_cmd_max>2</position_cmd_max>
+        <joint_name>arm_wrist_roll</joint_name><initial_position>0</initial_position>
+        <position_p_gain>12</position_p_gain><position_i_gain>0.1</position_i_gain><position_d_gain>0.4</position_d_gain>
+        <position_cmd_min>-2</position_cmd_min><position_cmd_max>2</position_cmd_max>
+        <joint_name>arm_gripper</joint_name><initial_position>0</initial_position>
+        <position_p_gain>8</position_p_gain><position_i_gain>0.05</position_i_gain><position_d_gain>0.25</position_d_gain>
+        <position_cmd_min>-1</position_cmd_min><position_cmd_max>1</position_cmd_max>
       </plugin>
     </gazebo>
@@ -120,5 +193,12 @@
       <sensor name="front_camera" type="camera">
         <topic>/camera/front</topic><gz_frame_id>front_camera_optical_frame</gz_frame_id><update_rate>20</update_rate><always_on>true</always_on>
-        <camera><horizontal_fov>1.0472</horizontal_fov><image><width>640</width><height>480</height><format>R8G8B8</format></image><clip><near>0.05</near><far>20</far></clip></camera>
+        <camera><horizontal_fov>1.0472</horizontal_fov><image><width>640</width><height>480</height><format>R8G8B8</format></image><clip><near>0.05</near><far>20</far></clip><noise><type>gaussian</type><mean>0</mean><stddev>0.007</stddev></noise></camera>
+      </sensor>
+      <!-- The depth stream is deliberately lower-rate and noisier than RGB.
+           launch/bringup adds a seeded delay/dropout stage before exposing its
+           point cloud to MoveIt's occupancy-map monitor. -->
+      <sensor name="front_depth" type="depth_camera">
+        <topic>/camera/depth</topic><gz_frame_id>front_camera_optical_frame</gz_frame_id><update_rate>10</update_rate><always_on>true</always_on>
+        <camera><horizontal_fov>1.0472</horizontal_fov><image><width>320</width><height>240</height><format>R_FLOAT32</format></image><clip><near>0.10</near><far>3.0</far></clip><noise><type>gaussian</type><mean>0</mean><stddev>0.012</stddev></noise></camera>
       </sensor>
     </gazebo>

File: urdf/lekiwi_cad.urdf (robot description, URDF)
Before this commit: robot LeKiwi, 45 links, 44 joints
Joints:
- joint arm_wrist_roll: limit (none) -> lower=-3.14159265359 upper=3.14159265359 effort=2 velocity=3

Commit message: feat: add Astra RGB-D deployment support

File: urdf/lekiwi.urdf.xacro (robot description, xacro)
@@ -36,4 +36,17 @@
   <joint name="front_camera_optical" type="fixed">
     <parent link="front_camera_link"/><child link="front_camera_optical_frame"/>
+    <origin xyz="0 0 0" rpy="-1.57079632679 0 -1.57079632679"/>
+  </joint>
+  <!-- Astra Pro is a third camera beside the existing front and wrist cameras.
+       Replace this measured mounting offset when its bracket is finalized;
+       camera drivers must not publish a competing runtime mount TF. -->
+  <link name="astra_camera_link"/>
+  <joint name="astra_camera_mount" type="fixed">
+    <parent link="front_camera_link"/><child link="astra_camera_link"/>
+    <origin xyz="0 0 0" rpy="0 0 0"/>
+  </joint>
+  <link name="astra_camera_optical_frame"/>
+  <joint name="astra_camera_optical" type="fixed">
+    <parent link="astra_camera_link"/><child link="astra_camera_optical_frame"/>
     <origin xyz="0 0 0" rpy="-1.57079632679 0 -1.57079632679"/>
   </joint>

Commit message: feat(urdf): model RobotSkin LD06 mount

File: urdf/lekiwi.urdf.xacro (robot description, xacro)
@@ -109,9 +109,18 @@
   <xacro:collision_sphere_proxy name="wrist_roll_servo_collision_proxy" parent="STS3215_03a_Wrist_Roll-v1" xyz="-0.0165 0.0160 -0.0101" radius="0.0335"/>
   <xacro:collision_sphere_proxy name="gripper_servo_collision_proxy" parent="STS3215_03a-v1-4" xyz="-0.0203 -0.0160 0.0101" radius="0.0335"/>
-  <!-- LD06 is an optional add-on, not part of the upstream CAD. -->
+  <!-- LD06 scan plane: the RobotSkin base puts it 90 mm forward, 70 mm right,
+       and 31.5 mm above base_link.  Keep this frame on the CAD body so its
+       pose cannot diverge from the rendered physical mount. -->
   <link name="laser"/>
   <joint name="laser_mount" type="fixed">
-    <parent link="base_link"/><child link="laser"/>
-    <origin xyz="0 0 0.220" rpy="0 0 0"/>
+    <parent link="ld06_body"/><child link="laser"/>
+    <origin xyz="0 0 0.0195" rpy="0 0 0"/>
+  </joint>
+  <link name="lidar_collision_proxy">
+    <collision><origin xyz="0 0 0.0195" rpy="0 0 0"/><geometry><cylinder radius="0.0245" length="0.039"/></geometry></collision>
+  </link>
+  <joint name="lidar_collision_proxy_mount" type="fixed">
+    <parent link="ld06_body"/><child link="lidar_collision_proxy"/>
+    <origin xyz="0 0 0" rpy="0 0 0"/>
   </joint>
   <!-- Gazebo-only contact and actuator model.  The CAD wheel meshes and their

File: urdf/lekiwi_cad.urdf (robot description, URDF)
Before this commit: robot LeKiwi, 45 links, 44 joints
Links:
- added link ld06_body; visual mesh filename=package://lekiwi_rmf/urdf/meshes/ld06_body.stl scale=0.001 0.001 0.001
- added link robotskin_lidar_mount; visual mesh filename=package://lekiwi_rmf/urdf/meshes/robotskin_lidar_mount.stl scale=0.001 0.001 0.001
Joints:
- added joint ld06_body: type fixed, parent robotskin_lidar_mount, child ld06_body, origin xyz=0.02 -0.005 0.012 rpy=0 0 0
- added joint robotskin_lidar_mount: type fixed, parent base_plate_layer1-v5, child robotskin_lidar_mount, origin xyz=0.05 0.095 0 rpy=0 0 0

Commit message: feat(lidar): expose scan-frame calibration

File: urdf/lekiwi.urdf.xacro (robot description, xacro)
@@ -3,4 +3,10 @@
 <robot xmlns:xacro="http://www.ros.org/wiki/xacro" name="lekiwi">
   <xacro:arg name="sim" default="false"/>
+  <!-- Measured correction from the CAD LD06 centre to the real scan centre.
+       Keep these at zero until an RViz wall-alignment check says otherwise. -->
+  <xacro:arg name="lidar_offset_x" default="0"/>
+  <xacro:arg name="lidar_offset_y" default="0"/>
+  <xacro:arg name="lidar_offset_z" default="0"/>
+  <xacro:arg name="lidar_offset_yaw" default="0"/>
   <!-- The simulator now drives the same six bounded joints as the hardware.
        Keep the joint type identical in both descriptions so a plan validated
@@ -110,10 +116,15 @@
   <xacro:collision_sphere_proxy name="gripper_servo_collision_proxy" parent="STS3215_03a-v1-4" xyz="-0.0203 -0.0160 0.0101" radius="0.0335"/>
   <!-- LD06 scan plane: the RobotSkin base puts it 90 mm forward, 70 mm right,
-       and 31.5 mm above base_link.  Keep this frame on the CAD body so its
-       pose cannot diverge from the rendered physical mount. -->
+       and 31.5 mm above base_link. The nominal frame stays on the CAD body;
+       the child is the small measured correction used by the scan. -->
+  <link name="laser_nominal"/>
+  <joint name="laser_nominal_mount" type="fixed">
+    <parent link="ld06_body"/><child link="laser_nominal"/>
+    <origin xyz="0 0 0.0195" rpy="0 0 0"/>
+  </joint>
   <link name="laser"/>
-  <joint name="laser_mount" type="fixed">
-    <parent link="ld06_body"/><child link="laser"/>
-    <origin xyz="0 0 0.0195" rpy="0 0 0"/>
+  <joint name="laser_calibration" type="fixed">
+    <parent link="laser_nominal"/><child link="laser"/>
+    <origin xyz="$(arg lidar_offset_x) $(arg lidar_offset_y) $(arg lidar_offset_z)" rpy="0 0 $(arg lidar_offset_yaw)"/>
   </joint>
   <link name="lidar_collision_proxy">

Commit message: refactor: centralize integration contracts

File: urdf/lekiwi.urdf.xacro (robot description, xacro)
@@ -16,6 +16,28 @@
        Declaring it continuous makes MoveIt discard the configured bounds. -->
   <xacro:property name="roll_joint" value="revolute"/>
-  <!-- Vendored from robotmindio/LeKiwi at efa608d; see urdf/README.md. -->
+  <!-- Vendored from robotmindio/LeKiwi; see urdf/README.md. -->
   <xacro:include filename="lekiwi_cad.urdf"/>
+  <!-- The RobotSkin mount and LD06 body are repository-owned integration
+       geometry, not part of the upstream LeKiwi CAD export. -->
+  <link name="robotskin_lidar_mount">
+    <visual name="robotskin_lidar_mount_visual">
+      <origin xyz="0 0 0" rpy="0 0 0"/>
+      <geometry><mesh filename="package://lekiwi_rmf/urdf/meshes/robotskin_lidar_mount.stl" scale="0.001 0.001 0.001"/></geometry>
+    </visual>
+  </link>
+  <link name="ld06_body">
+    <visual name="ld06_body_visual">
+      <origin xyz="0 0 0" rpy="0 0 0"/>
+      <geometry><mesh filename="package://lekiwi_rmf/urdf/meshes/ld06_body.stl" scale="0.001 0.001 0.001"/></geometry>
+    </visual>
+  </link>
+  <joint name="robotskin_lidar_mount_joint" type="fixed">
+    <origin xyz="0.05 0.095 0" rpy="0 0 0"/>
+    <parent link="base_plate_layer1-v5"/><child link="robotskin_lidar_mount"/>
+  </joint>
+  <joint name="ld06_body_mount" type="fixed">
+    <origin xyz="0.02 -0.005 0.012" rpy="0 0 0"/>
+    <parent link="robotskin_lidar_mount"/><child link="ld06_body"/>
+  </joint>
   <!-- CAD's root is the lower base plate. Its +Y is the physical forward
        direction, so yaw -90 degrees aligns it with REP-103 +X forward. -->

File: urdf/lekiwi_cad.urdf (robot description, URDF)
Before this commit: robot LeKiwi, 47 links, 46 joints
Links:
- removed link ld06_body
- removed link robotskin_lidar_mount
Joints:
- removed joint ld06_body
- removed joint robotskin_lidar_mount
