Commit message: feat: model LeKiwi with SO-101 arm

File: urdf/lekiwi.urdf.xacro (robot description, xacro)
@@ -9,4 +9,8 @@
   <xacro:arg name="lidar_offset_z" default="0"/>
   <xacro:arg name="lidar_offset_yaw" default="0"/>
+  <!-- The wrist camera mount varies between SO-101 kits. Measure these two
+       transforms before using wrist images for geometric perception. -->
+  <xacro:arg name="wrist_camera_xyz" default="0 0 0"/>
+  <xacro:arg name="wrist_camera_rpy" default="0 0 0"/>
   <!-- The simulator now drives the same six bounded joints as the hardware.
        Keep the joint type identical in both descriptions so a plan validated
@@ -16,5 +20,5 @@
        Declaring it continuous makes MoveIt discard the configured bounds. -->
   <xacro:property name="roll_joint" value="revolute"/>
-  <!-- Vendored from robotmindio/LeKiwi at efa608d; see urdf/README.md. -->
+  <!-- Complete model vendored from robotmindio/LeKiwi at 597e2da; see urdf/README.md. -->
   <xacro:include filename="lekiwi_cad.urdf"/>
   <!-- CAD's root is the lower base plate. Its +Y is the physical forward
@@ -59,6 +63,6 @@
   <link name="wrist_camera_link"/>
   <joint name="wrist_camera_mount" type="fixed">
-    <parent link="Camera-Model-v3-1"/><child link="wrist_camera_link"/>
-    <origin xyz="0 0 0" rpy="0 0 0"/>
+    <parent link="so101_gripper_link"/><child link="wrist_camera_link"/>
+    <origin xyz="$(arg wrist_camera_xyz)" rpy="$(arg wrist_camera_rpy)"/>
   </joint>
   <link name="wrist_camera_optical_frame"/>
@@ -72,6 +76,6 @@
   </link>
   <joint name="tool0_mount" type="fixed">
-    <parent link="Wrist_Roll_08c-v1"/><child link="tool0"/>
-    <origin xyz="0 0.040 0" rpy="0 0 0"/>
+    <parent link="so101_gripper_frame_link"/><child link="tool0"/>
+    <origin xyz="0 0 0" rpy="0 0 0"/>
   </joint>
   <!-- Low-poly self-collision proxies. These are deliberately attached to the
@@ -98,21 +102,14 @@
   </xacro:macro>
   <!-- Pedestal and camera are part of the manipulator's swept volume. -->
-  <xacro:collision_sphere_proxy name="arm_pedestal_collision_proxy" parent="Base_08q-v1" xyz="-0.0400 -0.0330 0.0358" radius="0.0783"/>
+  <xacro:collision_sphere_proxy name="arm_pedestal_collision_proxy" parent="so101_base_link" xyz="0.0168 0 0.0336" radius="0.0857"/>
   <xacro:collision_sphere_proxy name="front_camera_collision_proxy" parent="Camera-Model-v3" xyz="-0.0158 0.0114 -0.0114" radius="0.0332"/>
-  <!-- CAD-derived arm shell envelopes. -->
-  <xacro:collision_capsule_proxy name="shoulder_collision_proxy" parent="Rotation_Pitch_08i-v1" xyz="-0.0008 -0.0145 0.0041" rpy="0.0762 -0.3162 -1.5708" radius="0.0500" cylinder_length="0.0062"/>
-  <xacro:collision_capsule_proxy name="upper_arm_collision_proxy" parent="SO_ARM100_08k_116_Square-v1" xyz="-0.0218 -0.0590 -0.0044" rpy="3.1344 1.4654 1.5708" radius="0.0427" cylinder_length="0.0653"/>
-  <xacro:collision_capsule_proxy name="forearm_collision_proxy" parent="SO_ARM100_08k_Mirror-v1" xyz="-0.0218 0.0522 0.0113" rpy="3.1103 1.3717 1.5708" radius="0.0421" cylinder_length="0.0565"/>
-  <xacro:collision_sphere_proxy name="wrist_collision_proxy" parent="Wrist_Roll_Pitch_08i-v1" xyz="-0.0114 0.0081 -0.0179" radius="0.0564"/>
-  <xacro:collision_capsule_proxy name="roll_collision_proxy" parent="Wrist_Roll_08c-v1" xyz="0.0141 0.0209 -0.0445" rpy="0.2026 0.4555 -1.5708" radius="0.0431" cylinder_length="0.0307"/>
-  <xacro:collision_capsule_proxy name="gripper_collision_proxy" parent="Moving_Jaw_08d-v1" xyz="0.0007 0.0335 -0.0247" rpy="2.9993 -0.4467 1.5708" radius="0.0328" cylinder_length="0.0355"/>
-  <!-- Servo housings protrude beyond the link shells and need their own
-       envelopes to prevent a plan passing through a motor body. -->
-  <xacro:collision_sphere_proxy name="shoulder_pan_servo_collision_proxy" parent="STS3215_03a-v1" xyz="-0.0102 0.0163 -0.0203" radius="0.0337"/>
-  <xacro:collision_sphere_proxy name="shoulder_lift_servo_collision_proxy" parent="STS3215_03a-v1-1" xyz="0.0163 0.0103 -0.0203" radius="0.0337"/>
-  <xacro:collision_sphere_proxy name="elbow_servo_collision_proxy" parent="STS3215_03a-v1-2" xyz="0.0163 -0.0119 0.0193" radius="0.0337"/>
-  <xacro:collision_sphere_proxy name="wrist_flex_servo_collision_proxy" parent="STS3215_03a-v1-3" xyz="0.0163 -0.0217 0.0067" radius="0.0337"/>
-  <xacro:collision_sphere_proxy name="wrist_roll_servo_collision_proxy" parent="STS3215_03a_Wrist_Roll-v1" xyz="-0.0165 0.0160 -0.0101" radius="0.0335"/>
-  <xacro:collision_sphere_proxy name="gripper_servo_collision_proxy" parent="STS3215_03a-v1-4" xyz="-0.0203 -0.0160 0.0101" radius="0.0335"/>
+  <!-- SO-101 aggregate links already contain their servo housings. These
+       CAD-bounds-derived envelopes therefore cover each complete moving link. -->
+  <xacro:collision_capsule_proxy name="shoulder_collision_proxy" parent="so101_shoulder_link" xyz="-0.0192 0.0012 -0.0091" rpy="0 0 0" radius="0.0458" cylinder_length="0.0190"/>
+  <xacro:collision_capsule_proxy name="upper_arm_collision_proxy" parent="so101_upper_arm_link" xyz="-0.0591 -0.0131 0.0202" rpy="0 1.5708 0" radius="0.0460" cylinder_length="0.0502"/>
+  <xacro:collision_capsule_proxy name="forearm_collision_proxy" parent="so101_lower_arm_link" xyz="-0.0666 0.0035 0.0202" rpy="0 1.5708 0" radius="0.0411" cylinder_length="0.0749"/>
+  <xacro:collision_sphere_proxy name="wrist_collision_proxy" parent="so101_wrist_link" xyz="-0.0022 -0.0269 0.0222" radius="0.0569"/>
+  <xacro:collision_capsule_proxy name="roll_collision_proxy" parent="so101_gripper_link" xyz="-0.0024 -0.0020 -0.0517" rpy="0 0 0" radius="0.0459" cylinder_length="0.0136"/>
+  <xacro:collision_capsule_proxy name="gripper_collision_proxy" parent="so101_moving_jaw_link" xyz="-0.0012 -0.0360 0.0189" rpy="1.5708 0 0" radius="0.0305" cylinder_length="0.0310"/>
   <!-- LD06 scan plane: the RobotSkin base puts it 90 mm forward, 70 mm right,
        and 31.5 mm above base_link. The nominal frame stays on the CAD body;

File: urdf/lekiwi_cad.urdf (robot description, URDF)
Before this commit: robot LeKiwi, 47 links, 46 joints
Links:
- removed link Base_08q-v1
- removed link Camera-Model-v3-1
- removed link Moving_Jaw_08d-v1
- removed link Passive_Horn_01-v1
- removed link Rotation_Pitch_08i-v1
- removed link SO_ARM100_08k_116_Square-v1
- removed link SO_ARM100_08k_Asym_Mirror_Clip-v1
- removed link SO_ARM100_08k_Mirror-v1
- removed link STS3215_03a-v1
- removed link STS3215_03a-v1-1
- removed link STS3215_03a-v1-2
- removed link STS3215_03a-v1-3
- removed link STS3215_03a-v1-4
- removed link STS3215_03a_Wrist_Roll-v1
- removed link WaveShare_Mounting_Plate_01d-v1
- removed link Wrist-Camera-Mount-v11
- removed link Wrist_Roll_08c-v1
- removed link Wrist_Roll_Pitch_08i-v1
- added link so101_base_link, mass 0.147; visual mesh filename=package://lekiwi_rmf/urdf/meshes/so101/base_motor_holder_so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; visual mesh filename=package://lekiwi_rmf/urdf/meshes/so101/base_so101_v2.stl
- added link so101_gripper_frame_link
- added link so101_gripper_link, mass 0.087; visual mesh filename=package://lekiwi_rmf/urdf/meshes/so101/sts3215_03a_v1.stl; visual mesh filename=package://lekiwi_rmf/urdf/meshes/so101/wrist_roll_follower_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
- added link so101_lower_arm_link, mass 0.104; visual mesh filename=package://lekiwi_rmf/urdf/meshes/so101/motor_holder_so101_w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; visual mesh filename=package://lekiwi_rmf/urdf/meshes/so101/sts3215_03a_v1.stl
- added link so101_moving_jaw_link, mass 0.012; visual mesh filename=package://lekiwi_rmf/urdf/meshes/so101/moving_jaw_so101_v1.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
- added link so101_shoulder_link, mass 0.100006; visual mesh filename=package://lekiwi_rmf/urdf/meshes/so101/motor_holder_so101_b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; visual mesh filename=package://lekiwi_rmf/urdf/meshes/so101/rotation_pitch_so101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
- added link so101_upper_arm_link, mass 0.103; visual mesh filename=package://lekiwi_rmf/urdf/meshes/so101/sts3215_03a_v1.stl; visual mesh filename=package://lekiwi_rmf/urdf/meshes/so101/upper_arm_so101_v1.s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
- added link so101_wrist_link, mass 0.079; visual mesh filename=package://lekiwi_rmf/urdf/meshes/so101/sts3215_03a_no_horn_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; visual mesh filename=package://lekiwi_rmf/urdf/meshes/so101/wrist_roll_pitch_so1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
Joints:
- removed joint Base_08q-v1_Rigid-43
- removed joint Base_08q-v1_Rigid-44
- removed joint Base_08q-v1_Rigid-47
- removed joint Rotation_Pitch_08i-v1_Rigid-46
- removed joint Rotation_Pitch_08i-v1_Rigid-48
- removed joint SO_ARM100_08k_116_Square-v1_Rigid-50
- removed joint SO_ARM100_08k_Mirror-v1_Rigid-52
- removed joint Wrist-Camera-Mount-v11_Rigid-71
- removed joint Wrist_Roll_08c-v1_Rigid-56
- removed joint Wrist_Roll_08c-v1_Rigid-58
- removed joint Wrist_Roll_Pitch_08i-v1_Rigid-54
- removed joint base_plate_layer2-v3_Rigid-42
- removed joint ld06_body
- removed joint robotskin_lidar_mount
- added joint ld06_body_mount: type fixed, parent robotskin_lidar_mount, child ld06_body, origin xyz=0.02 -0.005 0.012 rpy=0 0 0
- added joint robotskin_lidar_mount_joint: type fixed, parent base_plate_layer1-v5, child robotskin_lidar_mount, origin xyz=0.05 0.095 0 rpy=0 0 0
- added joint so101_gripper_frame_joint: type fixed, parent so101_gripper_link, child so101_gripper_frame_link, origin xyz=-0.0079 -0.000218121 -0.0981274 rpy=0 3.14159 0, axis 0 0 0
- added joint so101_mount: type fixed, parent base_plate_layer2-v3, child so101_base_link, origin xyz=0.0388353 0.06714801 0.007 rpy=0 0 3.14159
- joint arm_elbow_flex: axis 1.0 0.0 0.0 -> 0 0 1; child SO_ARM100_08k_Mirror-v1 -> so101_lower_arm_link; limit lower=-1.75 upper=1.75 effort=4 velocity=2 -> lower=-1.69 upper=1.69 effort=4 velocity=2; origin xyz=0.0346 -0.013069710000000002 0.03178184000000002 rpy=-6.842277657836021e-49 -3.4512664603419266e-31 -1.3877787807814457e-17 -> xyz=-0.11257 -0.028 1.73763e-16 rpy=-3.63608e-16 8.74301e-16 1.5708; parent STS3215_03a-v1-2 -> so101_upper_arm_link
- joint arm_gripper: axis -2.74128770133849e-31 -0.9063079999999999 -0.422618 -> 0 0 1; child Moving_Jaw_08d-v1 -> so101_moving_jaw_link; limit lower=0 upper=1.57 effort=1 velocity=2 -> lower=-0.174533 upper=1.74533 effort=1 velocity=2; origin xyz=-0.032799999999999996 -0.023912249999999986 0.027026410000000018 rpy=-1.5707963267948968 3.944304526105059e-31 -1.9721522630525295e-31 -> xyz=0.0202 0.0188 -0.0234 rpy=1.5708 -5.24284e-08 -1.41553e-15; parent STS3215_03a-v1-4 -> so101_gripper_link
- joint arm_shoulder_lift: axis 1.0 0.0 0.0 -> 0 0 1; child SO_ARM100_08k_116_Square-v1 -> so101_upper_arm_link; limit lower=-1.75 upper=1.75 effort=4 velocity=2 -> lower=-1.74533 upper=1.74533 effort=4 velocity=2; origin xyz=0.0346 0.010249999999999987 -0.032799999999999975 rpy=3.141592653589793 1.7181275903033976e-32 -3.1373434374976504e-48 -> xyz=-0.0303992 -0.0182778 -0.0542 rpy=-1.5708 -1.5708 0; parent STS3215_03a-v1-1 -> so101_shoulder_link
- joint arm_shoulder_pan: axis -3.944304526105059e-31 3.944304526105059e-31 1.0 -> 0 0 1; child Rotation_Pitch_08i-v1 -> so101_shoulder_link; limit lower=-1.92 upper=1.92 effort=4 velocity=2 -> lower=-1.91986 upper=1.91986 effort=4 velocity=2; origin xyz=-0.010250000000000084 0.03459999999999999 -0.032799999999999996 rpy=1.5707963267948966 -2.781046729970605e-32 3.94430452610506e-31 -> xyz=0.0388353 -8.97657e-09 0.0624 rpy=3.14159 4.18253e-17 -3.14159; parent STS3215_03a-v1 -> so101_base_link
- joint arm_wrist_flex: axis 1.0 0.0 9.860761315262648e-32 -> 0 0 1; child Wrist_Roll_Pitch_08i-v1 -> so101_wrist_link; limit lower=-1.75 upper=1.75 effort=2 velocity=3 -> lower=-1.65806 upper=1.65806 effort=2 velocity=3; origin xyz=0.0346 -0.03408158 0.004398620000000015 rpy=3.1415926535897922 9.860761315262648e-32 -9.503163413661107e-47 -> xyz=-0.1349 0.0052 3.62355e-17 rpy=4.02456e-15 8.67362e-16 -1.5708; parent STS3215_03a-v1-3 -> so101_lower_arm_link
- joint arm_wrist_roll: axis 0.0 0.42261799999999994 -0.9063079999999999 -> 0 0 1; child Wrist_Roll_08c-v1 -> so101_gripper_link; limit lower=-3.14159265359 upper=3.14159265359 effort=2 velocity=3 -> lower=-2.74385 upper=2.84121 effort=2 velocity=3; origin xyz=-0.028999999999999998 0.00810632 0.006869499999999995 rpy=3.141592653589793 -0.0 0.0 -> xyz=5.55112e-17 -0.0611 0.0181 rpy=1.5708 0.0486795 3.14159; parent STS3215_03a_Wrist_Roll-v1 -> so101_wrist_link

Commit message: fix: make sensor model and services resilient

File: urdf/lekiwi.urdf.xacro (robot description, xacro)
@@ -3,14 +3,13 @@
 <robot xmlns:xacro="http://www.ros.org/wiki/xacro" name="lekiwi">
   <xacro:arg name="sim" default="false"/>
-  <!-- Measured correction from the CAD LD06 centre to the real scan centre.
-       Keep these at zero until an RViz wall-alignment check says otherwise. -->
-  <xacro:arg name="lidar_offset_x" default="0"/>
-  <xacro:arg name="lidar_offset_y" default="0"/>
-  <xacro:arg name="lidar_offset_z" default="0"/>
-  <xacro:arg name="lidar_offset_yaw" default="0"/>
-  <!-- The wrist camera mount varies between SO-101 kits. Measure these two
-       transforms before using wrist images for geometric perception. -->
-  <xacro:arg name="wrist_camera_xyz" default="0 0 0"/>
-  <xacro:arg name="wrist_camera_rpy" default="0 0 0"/>
+  <!-- The one tracked source for physical sensor calibration.  Every consumer
+       expands this Xacro (robot_state_publisher, MoveIt, and RViz), so changing
+       a measured value here cannot make their models disagree. -->
+  <xacro:property name="astra_mount_xyz" value="0 0 0"/>
+  <xacro:property name="astra_mount_rpy" value="0 0 0"/>
+  <xacro:property name="wrist_camera_xyz" value="0 0 0"/>
+  <xacro:property name="wrist_camera_rpy" value="0 0 0"/>
+  <xacro:property name="lidar_offset_xyz" value="0 0 0"/>
+  <xacro:property name="lidar_offset_yaw" value="0"/>
   <!-- The simulator now drives the same six bounded joints as the hardware.
        Keep the joint type identical in both descriptions so a plan validated
@@ -48,11 +47,16 @@
     <origin xyz="0 0 0" rpy="-1.57079632679 0 -1.57079632679"/>
   </joint>
-  <!-- Astra Pro is a third camera beside the existing front and wrist cameras.
-       Replace this measured mounting offset when its bracket is finalized;
-       camera drivers must not publish a competing runtime mount TF. -->
-  <link name="astra_camera_link"/>
+  <!-- Astra Pro is distinct from the existing front and wrist cameras. Its
+       165 x 48 x 40 mm body is visual-only; mount calibration remains above. -->
+  <link name="astra_camera_link">
+    <visual>
+      <origin xyz="-0.020 0 0" rpy="0 0 0"/>
+      <geometry><box size="0.040 0.165 0.048"/></geometry>
+      <material name="astra_body"><color rgba="0.08 0.18 0.25 1"/></material>
+    </visual>
+  </link>
   <joint name="astra_camera_mount" type="fixed">
-    <parent link="front_camera_link"/><child link="astra_camera_link"/>
-    <origin xyz="0 0 0" rpy="0 0 0"/>
+    <parent link="Camera-Model-v3"/><child link="astra_camera_link"/>
+    <origin xyz="${astra_mount_xyz}" rpy="${astra_mount_rpy}"/>
   </joint>
   <link name="astra_camera_optical_frame"/>
@@ -64,5 +68,5 @@
   <joint name="wrist_camera_mount" type="fixed">
     <parent link="so101_gripper_link"/><child link="wrist_camera_link"/>
-    <origin xyz="$(arg wrist_camera_xyz)" rpy="$(arg wrist_camera_rpy)"/>
+    <origin xyz="${wrist_camera_xyz}" rpy="${wrist_camera_rpy}"/>
   </joint>
   <link name="wrist_camera_optical_frame"/>
@@ -123,5 +127,5 @@
   <joint name="laser_calibration" type="fixed">
     <parent link="laser_nominal"/><child link="laser"/>
-    <origin xyz="$(arg lidar_offset_x) $(arg lidar_offset_y) $(arg lidar_offset_z)" rpy="0 0 $(arg lidar_offset_yaw)"/>
+    <origin xyz="${lidar_offset_xyz}" rpy="0 0 ${lidar_offset_yaw}"/>
   </joint>
   <link name="lidar_collision_proxy">

Commit message: fix: vendor aligned LeKiwi mounts

File: urdf/lekiwi.urdf.xacro (robot description, xacro)
@@ -3,9 +3,9 @@
 <robot xmlns:xacro="http://www.ros.org/wiki/xacro" name="lekiwi">
   <xacro:arg name="sim" default="false"/>
-  <!-- The one tracked source for physical sensor calibration.  Every consumer
-       expands this Xacro (robot_state_publisher, MoveIt, and RViz), so changing
-       a measured value here cannot make their models disagree. -->
-  <xacro:property name="astra_mount_xyz" value="0 0 0"/>
-  <xacro:property name="astra_mount_rpy" value="0 0 0"/>
+  <!-- The compact Astra mount's CAD contact plane is 15.5 mm high at -8 degrees.
+       Every consumer expands this Xacro (robot_state_publisher, MoveIt, and RViz),
+       so its fixed placement and measured wrist/lidar corrections stay aligned. -->
+  <xacro:property name="astra_mount_xyz" value="0 0 0.0155"/>
+  <xacro:property name="astra_mount_rpy" value="-0.13962634015954636 0 0"/>
   <xacro:property name="wrist_camera_xyz" value="0 0 0"/>
   <xacro:property name="wrist_camera_rpy" value="0 0 0"/>
@@ -19,5 +19,5 @@
        Declaring it continuous makes MoveIt discard the configured bounds. -->
   <xacro:property name="roll_joint" value="revolute"/>
-  <!-- Complete model vendored from robotmindio/LeKiwi at 597e2da; see urdf/README.md. -->
+  <!-- Complete model vendored from robotmindio/LeKiwi at 0595140; see urdf/README.md. -->
   <xacro:include filename="lekiwi_cad.urdf"/>
   <!-- CAD's root is the lower base plate. Its +Y is the physical forward
@@ -48,5 +48,5 @@
   </joint>
   <!-- Astra Pro is distinct from the existing front and wrist cameras. Its
-       165 x 48 x 40 mm body is visual-only; mount calibration remains above. -->
+       compact CAD mount owns placement; this 165 x 48 x 40 mm body is visual-only. -->
   <link name="astra_camera_link">
     <visual>
@@ -57,5 +57,5 @@
   </link>
   <joint name="astra_camera_mount" type="fixed">
-    <parent link="Camera-Model-v3"/><child link="astra_camera_link"/>
+    <parent link="astra_pro_compact_mount"/><child link="astra_camera_link"/>
     <origin xyz="${astra_mount_xyz}" rpy="${astra_mount_rpy}"/>
   </joint>
@@ -116,5 +116,5 @@
   <xacro:collision_capsule_proxy name="roll_collision_proxy" parent="so101_gripper_link" xyz="-0.0024 -0.0020 -0.0517" rpy="0 0 0" radius="0.0459" cylinder_length="0.0136"/>
   <xacro:collision_capsule_proxy name="gripper_collision_proxy" parent="so101_moving_jaw_link" xyz="-0.0012 -0.0360 0.0189" rpy="1.5708 0 0" radius="0.0305" cylinder_length="0.0310"/>
-  <!-- LD06 scan plane: the RobotSkin base puts it 90 mm forward, 70 mm right,
+  <!-- LD06 scan plane: the RobotSkin base puts it 75 mm forward, 75 mm right,
        and 31.5 mm above base_link. The nominal frame stays on the CAD body;
        the child is the small measured correction used by the scan. -->

File: urdf/lekiwi_cad.urdf (robot description, URDF)
Before this commit: robot LeKiwi, 37 links, 36 joints
Links:
- added link astra_pro_compact_mount; visual mesh filename=package://lekiwi_rmf/urdf/meshes/astra_pro_compact_mount.stl scale=0.001 0.001 0.001
Joints:
- added joint astra_pro_compact_mount_joint: type fixed, parent base_plate_layer1-v5, child astra_pro_compact_mount, origin xyz=0 0.08 0 rpy=0 0 0
- joint robotskin_lidar_mount_joint: origin xyz=0.05 0.095 0 rpy=0 0 0 -> xyz=0.055 0.08 0 rpy=0 0 0
- joint so101_mount: origin xyz=0.0388353 0.06714801 0.007 rpy=0 0 3.14159 -> xyz=0.04 0.08 0.007 rpy=0 0 0

Commit message: fix: align Astra frames and retain robot descriptions in RViz

File: urdf/lekiwi.urdf.xacro (robot description, xacro)
@@ -7,5 +7,7 @@
        so its fixed placement and measured wrist/lidar corrections stay aligned. -->
   <xacro:property name="astra_mount_xyz" value="0 0 0.0155"/>
-  <xacro:property name="astra_mount_rpy" value="-0.13962634015954636 0 0"/>
+  <!-- The saddle faces CAD +Y. Convert the camera's REP-103 +X to +Y,
+       then apply the saddle's downward pitch (Rx(-pitch) * Rz(pi/2)). -->
+  <xacro:property name="astra_mount_rpy" value="0 0.13962634015954636 1.5707963267948966"/>
   <xacro:property name="wrist_camera_xyz" value="0 0 0"/>
   <xacro:property name="wrist_camera_rpy" value="0 0 0"/>

Commit message: fix: integrate corrected robot model and raw SO-101 pose calibration

File: urdf/lekiwi.urdf.xacro (robot description, xacro)
@@ -10,4 +10,7 @@
        then apply the saddle's downward pitch (Rx(-pitch) * Rz(pi/2)). -->
   <xacro:property name="astra_mount_rpy" value="0 0.13962634015954636 1.5707963267948966"/>
+  <!-- Nominal front-face centre of the body envelope; measure the optical
+       centre on the installed camera and retain that correction here. -->
+  <xacro:property name="astra_optical_xyz" value="0.020 0 0.024"/>
   <xacro:property name="wrist_camera_xyz" value="0 0 0"/>
   <xacro:property name="wrist_camera_rpy" value="0 0 0"/>
@@ -21,5 +24,5 @@
        Declaring it continuous makes MoveIt discard the configured bounds. -->
   <xacro:property name="roll_joint" value="revolute"/>
-  <!-- Complete model vendored from robotmindio/LeKiwi at 0595140; see urdf/README.md. -->
+  <!-- Complete model vendored from robotmindio/LeKiwi; see model-source.json. -->
   <xacro:include filename="lekiwi_cad.urdf"/>
   <!-- CAD's root is the lower base plate. Its +Y is the physical forward
@@ -53,5 +56,5 @@
   <link name="astra_camera_link">
     <visual>
-      <origin xyz="-0.020 0 0" rpy="0 0 0"/>
+      <origin xyz="0 0 0.024" rpy="0 0 0"/>
       <geometry><box size="0.040 0.165 0.048"/></geometry>
       <material name="astra_body"><color rgba="0.08 0.18 0.25 1"/></material>
@@ -65,5 +68,5 @@
   <joint name="astra_camera_optical" type="fixed">
     <parent link="astra_camera_link"/><child link="astra_camera_optical_frame"/>
-    <origin xyz="0 0 0" rpy="-1.57079632679 0 -1.57079632679"/>
+    <origin xyz="${astra_optical_xyz}" rpy="-1.57079632679 0 -1.57079632679"/>
   </joint>
   <link name="wrist_camera_link"/>
@@ -119,5 +122,5 @@
   <xacro:collision_capsule_proxy name="gripper_collision_proxy" parent="so101_moving_jaw_link" xyz="-0.0012 -0.0360 0.0189" rpy="1.5708 0 0" radius="0.0305" cylinder_length="0.0310"/>
   <!-- LD06 scan plane: the RobotSkin base puts it 75 mm forward, 75 mm right,
-       and 31.5 mm above base_link. The nominal frame stays on the CAD body;
+       and 88.5 mm above base_link. The nominal frame stays on the CAD body;
        the child is the small measured correction used by the scan. -->
   <link name="laser_nominal"/>

File: urdf/lekiwi_cad.urdf (robot description, URDF)
Before this commit: robot LeKiwi, 38 links, 37 joints
Links:
- link so101_wrist_link: geometry visual mesh filename=package://lekiwi_rmf/urdf/meshes/so101/native_wrist_flex.stl; visual mesh filename=package://lekiwi_rmf/urdf/meshes/so101/sts3215_03a_no_horn_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
Joints:
- joint astra_pro_compact_mount_joint: origin xyz=0 0.08 0 rpy=0 0 0 -> xyz=0 0.08 0.007 rpy=0 0 0; parent base_plate_layer1-v5 -> base_plate_layer2-v3
- joint robotskin_lidar_mount_joint: origin xyz=0.055 0.08 0 rpy=0 0 0 -> xyz=0.055 0.08 0.007 rpy=0 0 0; parent base_plate_layer1-v5 -> base_plate_layer2-v3
- joint so101_mount: origin xyz=0.04 0.08 0.007 rpy=0 0 0 -> xyz=8.90955446603e-08 0.10598331 0.00699999999992 rpy=-2.65358979335e-06 -7.04151787851e-12 -1.57080265359
