Commit message: wip: qualify full sensor collision model and document measurement blockers

File: urdf/lekiwi.urdf.xacro (robot description, xacro)
@@ -13,4 +13,6 @@
        centre on the installed camera and retain that correction here. -->
   <xacro:property name="astra_optical_xyz" value="0.020 0 0.024"/>
+  <xacro:property name="astra_body_xyz" value="0 0 0.024"/>
+  <xacro:property name="astra_body_size" value="0.040 0.165 0.048"/>
   <xacro:property name="wrist_camera_xyz" value="0 0 0"/>
   <xacro:property name="wrist_camera_rpy" value="0 0 0"/>
@@ -53,11 +55,16 @@
   </joint>
   <!-- Astra Pro is distinct from the existing front and wrist cameras. Its
-       compact CAD mount owns placement; this 165 x 48 x 40 mm body is visual-only. -->
+       compact CAD mount owns placement; the body envelope also participates
+       in planning so the arm cannot pass through the camera. -->
   <link name="astra_camera_link">
     <visual>
-      <origin xyz="0 0 0.024" rpy="0 0 0"/>
-      <geometry><box size="0.040 0.165 0.048"/></geometry>
+      <origin xyz="${astra_body_xyz}" rpy="0 0 0"/>
+      <geometry><box size="${astra_body_size}"/></geometry>
       <material name="astra_body"><color rgba="0.08 0.18 0.25 1"/></material>
     </visual>
+    <collision>
+      <origin xyz="${astra_body_xyz}" rpy="0 0 0"/>
+      <geometry><box size="${astra_body_size}"/></geometry>
+    </collision>
   </link>
   <joint name="astra_camera_mount" type="fixed">
@@ -81,7 +88,5 @@
   </joint>
   <!-- Tool frame before the independently planned gripper joint. -->
-  <link name="tool0">
-    <collision><geometry><sphere radius="0.025"/></geometry></collision>
-  </link>
+  <link name="tool0"/>
   <joint name="tool0_mount" type="fixed">
     <parent link="so101_gripper_frame_link"/><child link="tool0"/>
@@ -118,5 +123,13 @@
   <xacro:collision_capsule_proxy name="upper_arm_collision_proxy" parent="so101_upper_arm_link" xyz="-0.0591 -0.0131 0.0202" rpy="0 1.5708 0" radius="0.0460" cylinder_length="0.0502"/>
   <xacro:collision_capsule_proxy name="forearm_collision_proxy" parent="so101_lower_arm_link" xyz="-0.0666 0.0035 0.0202" rpy="0 1.5708 0" radius="0.0411" cylinder_length="0.0749"/>
-  <xacro:collision_sphere_proxy name="wrist_collision_proxy" parent="so101_wrist_link" xyz="-0.0022 -0.0269 0.0222" radius="0.0569"/>
+  <!-- Native wrist bounds plus 4 mm on each face. The old enclosing sphere
+       extended into the moving jaw even in the reference pose. -->
+  <link name="wrist_collision_proxy">
+    <collision><geometry><box size="0.04335 0.08584 0.07031"/></geometry></collision>
+  </link>
+  <joint name="wrist_collision_proxy_mount" type="fixed">
+    <parent link="so101_wrist_link"/><child link="wrist_collision_proxy"/>
+    <origin xyz="-0.00233 -0.026915 0.02215"/>
+  </joint>
   <xacro:collision_capsule_proxy name="roll_collision_proxy" parent="so101_gripper_link" xyz="-0.0024 -0.0020 -0.0517" rpy="0 0 0" radius="0.0459" cylinder_length="0.0136"/>
   <xacro:collision_capsule_proxy name="gripper_collision_proxy" parent="so101_moving_jaw_link" xyz="-0.0012 -0.0360 0.0189" rpy="1.5708 0 0" radius="0.0305" cylinder_length="0.0310"/>

Commit message: fix: integrate outward arm and rear Pi-hole lidar placement

File: urdf/lekiwi.urdf.xacro (robot description, xacro)
@@ -134,5 +134,6 @@
   <xacro:collision_capsule_proxy name="roll_collision_proxy" parent="so101_gripper_link" xyz="-0.0024 -0.0020 -0.0517" rpy="0 0 0" radius="0.0459" cylinder_length="0.0136"/>
   <xacro:collision_capsule_proxy name="gripper_collision_proxy" parent="so101_moving_jaw_link" xyz="-0.0012 -0.0360 0.0189" rpy="1.5708 0 0" radius="0.0305" cylinder_length="0.0310"/>
-  <!-- LD06 scan plane: the RobotSkin base puts it 75 mm forward, 75 mm right,
+  <!-- LD06 scan plane: the rear Pi-hole-mounted RobotSkin base puts it
+       135 mm behind the origin, 5 mm left,
        and 88.5 mm above base_link. The nominal frame stays on the CAD body;
        the child is the small measured correction used by the scan. -->

File: urdf/lekiwi_cad.urdf (robot description, URDF)
Before this commit: robot LeKiwi, 38 links, 37 joints
Links:
- removed link Bottom-V2-v3
- removed link Top-V2-v2
Joints:
- removed joint Bottom-V2-v3_Rigid-24
- removed joint base_plate_layer2-v3_Rigid-22
- joint robotskin_lidar_mount_joint: origin xyz=0.055 0.08 0.007 rpy=0 0 0 -> xyz=0.0 -0.115 0.007 rpy=0 0 -1.5707963267948966
- joint so101_mount: origin xyz=8.90955446603e-08 0.10598331 0.00699999999992 rpy=-2.65358979335e-06 -7.04151787851e-12 -1.57080265359 -> xyz=-8.90955448261e-08 0.0283127100002 0.00699999999992 rpy=-2.65358979335e-06 -7.04151787872e-12 1.57079

Commit message: fix: integrate Astra on operator-selected left mounting holes

File: urdf/lekiwi.urdf.xacro (robot description, xacro)
@@ -7,5 +7,5 @@
        so its fixed placement and measured wrist/lidar corrections stay aligned. -->
   <xacro:property name="astra_mount_xyz" value="0 0 0.0155"/>
-  <!-- The saddle faces CAD +Y. Convert the camera's REP-103 +X to +Y,
+  <!-- The saddle faces its local +Y. Convert the camera's REP-103 +X to +Y,
        then apply the saddle's downward pitch (Rx(-pitch) * Rz(pi/2)). -->
   <xacro:property name="astra_mount_rpy" value="0 0.13962634015954636 1.5707963267948966"/>

File: urdf/lekiwi_cad.urdf (robot description, URDF)
Before this commit: robot LeKiwi, 36 links, 35 joints
Joints:
- joint astra_pro_compact_mount_joint: origin xyz=0 0.08 0.007 rpy=0 0 0 -> xyz=-0.1 0 0.007 rpy=0 0 1.5707963267948966

Commit message: Fix model generation and simulation consistency

File: urdf/lekiwi.urdf.xacro (robot description, xacro)
@@ -47,5 +47,7 @@
   <joint name="front_camera_mount" type="fixed">
     <parent link="Camera-Model-v3"/><child link="front_camera_link"/>
-    <origin xyz="0 0 0" rpy="0 0 0"/>
+    <!-- The CAD camera PCB faces local +Y; make that the ROS camera-link +X
+         while retaining the board's measured roll around the lens axis. -->
+    <origin xyz="0 0 0" rpy="1.57079632679 0 1.57079632679"/>
   </joint>
   <link name="front_camera_optical_frame"/>
@@ -200,6 +202,6 @@
       <!-- Gazebo-native fail-safe: public bridge topics are forwarded only
            while fresh. If ros_gz_bridge or either ROS adapter disappears,
-           it actively zeros wheel demand and interrupts the native arm
-           trajectory with a current-position hold. -->
+           it actively zeros wheel demand and holds the arm at its current
+           position. -->
       <plugin filename="liblekiwi_sim_native_failsafe.so" name="lekiwi_rmf::SimNativeFailsafe"/>
       <plugin filename="gz-sim-joint-state-publisher-system" name="gz::sim::systems::JointStatePublisher">
@@ -215,29 +217,32 @@
         <joint_name>arm_gripper</joint_name>
       </plugin>
-      <plugin filename="gz-sim-joint-trajectory-controller-system" name="gz::sim::systems::JointTrajectoryController">
-        <topic>/sim/arm/native_joint_trajectory</topic>
-        <joint_name>arm_shoulder_pan</joint_name><initial_position>0</initial_position>
-        <position_p_gain>18</position_p_gain><position_i_gain>0.2</position_i_gain><position_d_gain>0.8</position_d_gain>
-        <position_cmd_min>-4</position_cmd_min><position_cmd_max>4</position_cmd_max>
-        <joint_name>arm_shoulder_lift</joint_name><initial_position>0</initial_position>
-        <position_p_gain>70</position_p_gain><position_i_gain>0.3</position_i_gain><position_d_gain>2.0</position_d_gain>
-        <position_cmd_min>-4</position_cmd_min><position_cmd_max>4</position_cmd_max>
-        <joint_name>arm_elbow_flex</joint_name><initial_position>0</initial_position>
-        <position_p_gain>70</position_p_gain><position_i_gain>0.3</position_i_gain><position_d_gain>2.0</position_d_gain>
-        <position_cmd_min>-4</position_cmd_min><position_cmd_max>4</position_cmd_max>
-        <joint_name>arm_wrist_flex</joint_name><initial_position>0</initial_position>
-        <position_p_gain>12</position_p_gain><position_i_gain>0.1</position_i_gain><position_d_gain>0.4</position_d_gain>
-        <position_cmd_min>-2</position_cmd_min><position_cmd_max>2</position_cmd_max>
-        <joint_name>arm_wrist_roll</joint_name><initial_position>0</initial_position>
-        <position_p_gain>12</position_p_gain><position_i_gain>0.1</position_i_gain><position_d_gain>0.4</position_d_gain>
-        <position_cmd_min>-2</position_cmd_min><position_cmd_max>2</position_cmd_max>
-        <joint_name>arm_gripper</joint_name><initial_position>0</initial_position>
-        <position_p_gain>8</position_p_gain><position_i_gain>0.05</position_i_gain><position_d_gain>0.25</position_d_gain>
-        <position_cmd_min>-1</position_cmd_min><position_cmd_max>1</position_cmd_max>
+      <plugin filename="gz-sim-joint-position-controller-system" name="gz::sim::systems::JointPositionController">
+        <joint_name>arm_shoulder_pan</joint_name><topic>/sim/arm/arm_shoulder_pan/native_cmd_pos</topic><initial_position>0</initial_position>
+        <p_gain>18</p_gain><i_gain>0.2</i_gain><d_gain>0.8</d_gain><cmd_min>-4</cmd_min><cmd_max>4</cmd_max>
+      </plugin>
+      <plugin filename="gz-sim-joint-position-controller-system" name="gz::sim::systems::JointPositionController">
+        <joint_name>arm_shoulder_lift</joint_name><topic>/sim/arm/arm_shoulder_lift/native_cmd_pos</topic><initial_position>0</initial_position>
+        <p_gain>70</p_gain><i_gain>0.3</i_gain><d_gain>2.0</d_gain><cmd_min>-4</cmd_min><cmd_max>4</cmd_max>
+      </plugin>
+      <plugin filename="gz-sim-joint-position-controller-system" name="gz::sim::systems::JointPositionController">
+        <joint_name>arm_elbow_flex</joint_name><topic>/sim/arm/arm_elbow_flex/native_cmd_pos</topic><initial_position>0</initial_position>
+        <p_gain>70</p_gain><i_gain>0.3</i_gain><d_gain>2.0</d_gain><cmd_min>-4</cmd_min><cmd_max>4</cmd_max>
+      </plugin>
+      <plugin filename="gz-sim-joint-position-controller-system" name="gz::sim::systems::JointPositionController">
+        <joint_name>arm_wrist_flex</joint_name><topic>/sim/arm/arm_wrist_flex/native_cmd_pos</topic><initial_position>0</initial_position>
+        <p_gain>12</p_gain><i_gain>0.1</i_gain><d_gain>0.4</d_gain><cmd_min>-2</cmd_min><cmd_max>2</cmd_max>
+      </plugin>
+      <plugin filename="gz-sim-joint-position-controller-system" name="gz::sim::systems::JointPositionController">
+        <joint_name>arm_wrist_roll</joint_name><topic>/sim/arm/arm_wrist_roll/native_cmd_pos</topic><initial_position>0</initial_position>
+        <p_gain>12</p_gain><i_gain>0.1</i_gain><d_gain>0.4</d_gain><cmd_min>-2</cmd_min><cmd_max>2</cmd_max>
+      </plugin>
+      <plugin filename="gz-sim-joint-position-controller-system" name="gz::sim::systems::JointPositionController">
+        <joint_name>arm_gripper</joint_name><topic>/sim/arm/arm_gripper/native_cmd_pos</topic><initial_position>0</initial_position>
+        <p_gain>8</p_gain><i_gain>0.05</i_gain><d_gain>0.25</d_gain><cmd_min>-1</cmd_min><cmd_max>1</cmd_max>
       </plugin>
     </gazebo>
     <gazebo reference="laser">
       <sensor name="lidar" type="gpu_lidar">
-        <topic>/scan</topic><gz_frame_id>laser</gz_frame_id><update_rate>10</update_rate><always_on>true</always_on>
+        <topic>/scan</topic><update_rate>10</update_rate><always_on>true</always_on>
         <lidar><scan><horizontal><samples>360</samples><resolution>1</resolution><min_angle>-3.14159</min_angle><max_angle>3.14159</max_angle></horizontal></scan><range><min>0.08</min><max>12</max><resolution>0.01</resolution></range></lidar>
       </sensor>
@@ -245,5 +250,5 @@
     <gazebo reference="front_camera_link">
       <sensor name="front_camera" type="camera">
-        <topic>/camera/front</topic><gz_frame_id>front_camera_optical_frame</gz_frame_id><update_rate>20</update_rate><always_on>true</always_on>
+        <topic>/camera/front</topic><update_rate>20</update_rate><always_on>true</always_on>
         <camera><horizontal_fov>1.0472</horizontal_fov><image><width>640</width><height>480</height><format>R8G8B8</format></image><clip><near>0.05</near><far>20</far></clip><noise><type>gaussian</type><mean>0</mean><stddev>0.007</stddev></noise></camera>
       </sensor>
@@ -252,5 +257,5 @@
            point cloud to MoveIt's occupancy-map monitor. -->
       <sensor name="front_depth" type="depth_camera">
-        <topic>/camera/depth</topic><gz_frame_id>front_camera_optical_frame</gz_frame_id><update_rate>10</update_rate><always_on>true</always_on>
+        <topic>/camera/depth</topic><update_rate>10</update_rate><always_on>true</always_on>
         <camera><horizontal_fov>1.0472</horizontal_fov><image><width>320</width><height>240</height><format>R_FLOAT32</format></image><clip><near>0.10</near><far>3.0</far></clip><noise><type>gaussian</type><mean>0</mean><stddev>0.012</stddev></noise></camera>
       </sensor>

Commit message: fix: use CAD meshes for arm collision proxies

File: urdf/lekiwi.urdf.xacro (robot description, xacro)
@@ -95,10 +95,6 @@
     <origin xyz="0 0 0" rpy="0 0 0"/>
   </joint>
-  <!-- Low-poly self-collision proxies. These are deliberately attached to the
-       CAD links, so their kinematics remain exact while planning stays
-       real-time.  The dimensions below enclose the vendored mesh bounding
-       vertices with a further 4 mm clearance; they are not substitute visual
-       geometry.  A capsule is a cylinder along local Z with a sphere on each
-       end, which covers a complete arm link instead of just its joint centre. -->
+  <!-- Collision proxies stay attached to their CAD links. Prefer exact
+       vendored meshes where enclosing primitives create false collisions. -->
   <xacro:macro name="collision_sphere_proxy" params="name parent xyz radius">
     <link name="${name}"><collision><geometry><sphere radius="${radius}"/></geometry></collision></link>
@@ -117,11 +113,26 @@
     </joint>
   </xacro:macro>
-  <!-- Pedestal and camera are part of the manipulator's swept volume. -->
-  <xacro:collision_sphere_proxy name="arm_pedestal_collision_proxy" parent="so101_base_link" xyz="0.0168 0 0.0336" radius="0.0857"/>
+  <!-- Exact CAD collision meshes avoid the pedestal sphere/upper-arm capsule
+       overlapping in poses where the physical parts are separated. -->
+  <link name="arm_pedestal_collision_proxy">
+    <collision><origin xyz="-0.00636471 -9.94414e-05 -0.0024" rpy="1.5708 -1.67685e-15 1.5708"/><geometry><mesh filename="package://lekiwi_rmf/urdf/meshes/so101/base_motor_holder_so101_v1.stl"/></geometry></collision>
+    <collision><origin xyz="-0.00636471 -8.97657e-09 -0.0024" rpy="1.5708 -2.78073e-29 1.5708"/><geometry><mesh filename="package://lekiwi_rmf/urdf/meshes/so101/base_so101_v2.stl"/></geometry></collision>
+    <collision><origin xyz="0.0263353 -8.97657e-09 0.0437" rpy="-8.21148e-16 7.84513e-18 1.249e-15"/><geometry><mesh filename="package://lekiwi_rmf/urdf/meshes/so101/sts3215_03a_v1.stl"/></geometry></collision>
+    <collision><origin xyz="-0.0309827 -0.000199441 0.0474" rpy="1.5708 -1.35493e-14 1.5708"/><geometry><mesh filename="package://lekiwi_rmf/urdf/meshes/so101/waveshare_mounting_plate_so101_v2.stl"/></geometry></collision>
+  </link>
+  <joint name="arm_pedestal_collision_proxy_mount" type="fixed">
+    <parent link="so101_base_link"/><child link="arm_pedestal_collision_proxy"/><origin xyz="0 0 0" rpy="0 0 0"/>
+  </joint>
   <xacro:collision_sphere_proxy name="front_camera_collision_proxy" parent="Camera-Model-v3" xyz="-0.0158 0.0114 -0.0114" radius="0.0332"/>
   <!-- SO-101 aggregate links already contain their servo housings. These
        CAD-bounds-derived envelopes therefore cover each complete moving link. -->
   <xacro:collision_capsule_proxy name="shoulder_collision_proxy" parent="so101_shoulder_link" xyz="-0.0192 0.0012 -0.0091" rpy="0 0 0" radius="0.0458" cylinder_length="0.0190"/>
-  <xacro:collision_capsule_proxy name="upper_arm_collision_proxy" parent="so101_upper_arm_link" xyz="-0.0591 -0.0131 0.0202" rpy="0 1.5708 0" radius="0.0460" cylinder_length="0.0502"/>
+  <link name="upper_arm_collision_proxy">
+    <collision><origin xyz="-0.11257 -0.0155 0.0187" rpy="-3.14159 -5.27356e-16 -1.5708"/><geometry><mesh filename="package://lekiwi_rmf/urdf/meshes/so101/sts3215_03a_v1.stl"/></geometry></collision>
+    <collision><origin xyz="-0.065085 0.012 0.0182" rpy="3.14159 -0 -1.30911e-30"/><geometry><mesh filename="package://lekiwi_rmf/urdf/meshes/so101/upper_arm_so101_v1.stl"/></geometry></collision>
+  </link>
+  <joint name="upper_arm_collision_proxy_mount" type="fixed">
+    <parent link="so101_upper_arm_link"/><child link="upper_arm_collision_proxy"/><origin xyz="0 0 0" rpy="0 0 0"/>
+  </joint>
   <xacro:collision_capsule_proxy name="forearm_collision_proxy" parent="so101_lower_arm_link" xyz="-0.0666 0.0035 0.0202" rpy="0 1.5708 0" radius="0.0411" cylinder_length="0.0749"/>
   <!-- Native wrist bounds plus 4 mm on each face. The old enclosing sphere

Commit message: fix: align MoveIt with calibrated gripper and stow

File: urdf/lekiwi.urdf.xacro (robot description, xacro)
@@ -38,4 +38,15 @@
     <parent link="base_footprint"/><child link="base_link"/>
     <origin xyz="0 0 0.093" rpy="0 0 0"/>
+  </joint>
+  <!-- Distal arm links stay outside the vertical airspace above the chassis.
+       The radius and lower plane come from the base collision model. -->
+  <link name="arm_workspace_keepout_proxy">
+    <xacro:unless value="$(arg sim)">
+      <collision><geometry><cylinder radius="0.145" length="0.650"/></geometry></collision>
+    </xacro:unless>
+  </link>
+  <joint name="arm_workspace_keepout_mount" type="fixed">
+    <parent link="base_footprint"/><child link="arm_workspace_keepout_proxy"/>
+    <origin xyz="0 0 0.463" rpy="0 0 0"/>
   </joint>
   <joint name="base_link_to_cad" type="fixed">

Commit message: fix: add a ground keepout for arm planning

File: urdf/lekiwi.urdf.xacro (robot description, xacro)
@@ -38,4 +38,18 @@
     <parent link="base_footprint"/><child link="base_link"/>
     <origin xyz="0 0 0.093" rpy="0 0 0"/>
+  </joint>
+  <!-- base_footprint is the floor-contact plane on the level physical robot.
+       A live depth cloud is not a reliable substitute for this hard arm limit. -->
+  <link name="arm_ground_keepout_proxy">
+    <xacro:unless value="$(arg sim)">
+      <collision>
+        <origin xyz="0 0 -0.01"/>
+        <geometry><box size="2.0 2.0 0.02"/></geometry>
+      </collision>
+    </xacro:unless>
+  </link>
+  <joint name="arm_ground_keepout_mount" type="fixed">
+    <parent link="base_footprint"/><child link="arm_ground_keepout_proxy"/>
+    <origin xyz="0 0 0" rpy="0 0 0"/>
   </joint>
   <!-- Distal arm links stay outside the vertical airspace above the chassis.

Commit message: fix: cover the full arm volume below floor

File: urdf/lekiwi.urdf.xacro (robot description, xacro)
@@ -44,6 +44,6 @@
     <xacro:unless value="$(arg sim)">
       <collision>
-        <origin xyz="0 0 -0.01"/>
-        <geometry><box size="2.0 2.0 0.02"/></geometry>
+        <origin xyz="0 0 -1.0"/>
+        <geometry><box size="2.0 2.0 2.0"/></geometry>
       </collision>
     </xacro:unless>

Commit message: fix: enforce arm floor clearance and lighten bus polling

File: urdf/lekiwi.urdf.xacro (robot description, xacro)
@@ -39,10 +39,11 @@
     <origin xyz="0 0 0.093" rpy="0 0 0"/>
   </joint>
-  <!-- base_footprint is the floor-contact plane on the level physical robot.
-       A live depth cloud is not a reliable substitute for this hard arm limit. -->
+  <!-- Keep arm collision geometry 20 mm above the wheel-contact plane. The
+       nominal CAD plane admitted a physically floor-touching pose, so this
+       margin covers the observed model-to-hardware offset. -->
   <link name="arm_ground_keepout_proxy">
     <xacro:unless value="$(arg sim)">
       <collision>
-        <origin xyz="0 0 -1.0"/>
+        <origin xyz="0 0 -0.98"/>
         <geometry><box size="2.0 2.0 2.0"/></geometry>
       </collision>

Commit message: fix: model wrist roll collision with CAD meshes

File: urdf/lekiwi.urdf.xacro (robot description, xacro)
@@ -171,5 +171,11 @@
     <origin xyz="-0.00233 -0.026915 0.02215"/>
   </joint>
-  <xacro:collision_capsule_proxy name="roll_collision_proxy" parent="so101_gripper_link" xyz="-0.0024 -0.0020 -0.0517" rpy="0 0 0" radius="0.0459" cylinder_length="0.0136"/>
+  <link name="roll_collision_proxy">
+    <collision><origin xyz="0.0077 0.0001 -0.0234" rpy="-1.5708 -5.19179e-17 -1.66533e-16"/><geometry><mesh filename="package://lekiwi_rmf/urdf/meshes/so101/sts3215_03a_v1.stl"/></geometry></collision>
+    <collision><origin xyz="8.32667e-17 -0.000218214 0.000949706" rpy="-3.14159 -5.55112e-17 0"/><geometry><mesh filename="package://lekiwi_rmf/urdf/meshes/so101/wrist_roll_follower_so101_v1.stl"/></geometry></collision>
+  </link>
+  <joint name="roll_collision_proxy_mount" type="fixed">
+    <parent link="so101_gripper_link"/><child link="roll_collision_proxy"/>
+  </joint>
   <xacro:collision_capsule_proxy name="gripper_collision_proxy" parent="so101_moving_jaw_link" xyz="-0.0012 -0.0360 0.0189" rpy="1.5708 0 0" radius="0.0305" cylinder_length="0.0310"/>
   <!-- LD06 scan plane: the rear Pi-hole-mounted RobotSkin base puts it
