Commit message: fix: match arm keepouts to physical chassis and floor

File: urdf/lekiwi.urdf.xacro (robot description, xacro)
@@ -39,11 +39,10 @@
     <origin xyz="0 0 0.093" rpy="0 0 0"/>
   </joint>
-  <!-- Keep arm collision geometry 20 mm above the wheel-contact plane. The
-       nominal CAD plane admitted a physically floor-touching pose, so this
-       margin covers the observed model-to-hardware offset. -->
+  <!-- The wheel-contact plane is the floor. Keep modeled parts above it while
+       allowing the gripper to approach objects lying on the floor. -->
   <link name="arm_ground_keepout_proxy">
     <xacro:unless value="$(arg sim)">
       <collision>
-        <origin xyz="0 0 -0.98"/>
+        <origin xyz="0 0 -1.0"/>
         <geometry><box size="2.0 2.0 2.0"/></geometry>
       </collision>
@@ -53,15 +52,4 @@
     <parent link="base_footprint"/><child link="arm_ground_keepout_proxy"/>
     <origin xyz="0 0 0" rpy="0 0 0"/>
-  </joint>
-  <!-- Distal arm links stay outside the vertical airspace above the chassis.
-       The radius and lower plane come from the base collision model. -->
-  <link name="arm_workspace_keepout_proxy">
-    <xacro:unless value="$(arg sim)">
-      <collision><geometry><cylinder radius="0.145" length="0.650"/></geometry></collision>
-    </xacro:unless>
-  </link>
-  <joint name="arm_workspace_keepout_mount" type="fixed">
-    <parent link="base_footprint"/><child link="arm_workspace_keepout_proxy"/>
-    <origin xyz="0 0 0.463" rpy="0 0 0"/>
   </joint>
   <joint name="base_link_to_cad" type="fixed">
@@ -178,5 +166,10 @@
     <parent link="so101_gripper_link"/><child link="roll_collision_proxy"/>
   </joint>
-  <xacro:collision_capsule_proxy name="gripper_collision_proxy" parent="so101_moving_jaw_link" xyz="-0.0012 -0.0360 0.0189" rpy="1.5708 0 0" radius="0.0305" cylinder_length="0.0310"/>
+  <link name="gripper_collision_proxy">
+    <collision><origin xyz="-5.55112e-17 -5.55112e-17 0.0189" rpy="9.53145e-17 6.93889e-18 1.24077e-24"/><geometry><mesh filename="package://lekiwi_rmf/urdf/meshes/so101/moving_jaw_so101_v1.stl"/></geometry></collision>
+  </link>
+  <joint name="gripper_collision_proxy_mount" type="fixed">
+    <parent link="so101_moving_jaw_link"/><child link="gripper_collision_proxy"/>
+  </joint>
   <!-- LD06 scan plane: the rear Pi-hole-mounted RobotSkin base puts it
        135 mm behind the origin, 5 mm left,

Commit message: fix: align LD06 scan with Astra landmark

File: urdf/lekiwi.urdf.xacro (robot description, xacro)
@@ -18,5 +18,7 @@
   <xacro:property name="wrist_camera_rpy" value="0 0 0"/>
   <xacro:property name="lidar_offset_xyz" value="0 0 0"/>
-  <xacro:property name="lidar_offset_yaw" value="0"/>
+  <!-- A shared bottle landmark in the LD06 scan and Astra cloud measured a
+       90-degree clockwise correction to the nominal CAD scan axis. -->
+  <xacro:property name="lidar_offset_yaw" value="-1.5707963267948966"/>
   <!-- The simulator now drives the same six bounded joints as the hardware.
        Keep the joint type identical in both descriptions so a plan validated

Commit message: fix: shape and display chassis collision guard

File: urdf/lekiwi.urdf.xacro (robot description, xacro)
@@ -34,6 +34,17 @@
   <link name="base_footprint"/>
   <link name="base_link">
-    <!-- Conservative planning proxy; CAD meshes are visual-only. -->
-    <collision><geometry><cylinder radius="0.145" length="0.090"/></geometry></collision>
+    <!-- Keep only the rear of the chassis guard. Its front cut is tangent to
+         the center-facing edge of the arm pedestal; the lower face stays at
+         z=48 mm above the floor, with a 50 mm height. -->
+    <collision>
+      <origin xyz="0 0 -0.020"/>
+      <geometry><mesh filename="package://lekiwi_rmf/urdf/chassis_guard.stl"/></geometry>
+    </collision>
+    <!-- Show the exact restricted volume in the default RViz RobotModel. -->
+    <visual>
+      <origin xyz="0 0 -0.020"/>
+      <geometry><mesh filename="package://lekiwi_rmf/urdf/chassis_guard.stl"/></geometry>
+      <material name="chassis_guard"><color rgba="1 0.2 0.1 0.5"/></material>
+    </visual>
   </link>
   <joint name="base_footprint_to_base_link" type="fixed">

Commit message: fix: use physical front camera geometry for resting arm recovery

File: urdf/lekiwi.urdf.xacro (robot description, xacro)
@@ -124,10 +124,4 @@
   <!-- Collision proxies stay attached to their CAD links. Prefer exact
        vendored meshes where enclosing primitives create false collisions. -->
-  <xacro:macro name="collision_sphere_proxy" params="name parent xyz radius">
-    <link name="${name}"><collision><geometry><sphere radius="${radius}"/></geometry></collision></link>
-    <joint name="${name}_mount" type="fixed">
-      <parent link="${parent}"/><child link="${name}"/><origin xyz="${xyz}" rpy="0 0 0"/>
-    </joint>
-  </xacro:macro>
   <xacro:macro name="collision_capsule_proxy" params="name parent xyz rpy radius cylinder_length">
     <link name="${name}">
@@ -151,5 +145,12 @@
     <parent link="so101_base_link"/><child link="arm_pedestal_collision_proxy"/><origin xyz="0 0 0" rpy="0 0 0"/>
   </joint>
-  <xacro:collision_sphere_proxy name="front_camera_collision_proxy" parent="Camera-Model-v3" xyz="-0.0158 0.0114 -0.0114" radius="0.0332"/>
+  <!-- The enclosing camera sphere reached into the wrist at a valid resting
+       pose. Use the physical camera mesh while retaining collision checking. -->
+  <link name="front_camera_collision_proxy">
+    <collision><origin xyz="0 0 0" rpy="0 0 0"/><geometry><mesh filename="package://lekiwi_rmf/urdf/meshes/Camera-Model-v3.stl" scale="0.001 0.001 0.001"/></geometry></collision>
+  </link>
+  <joint name="front_camera_collision_proxy_mount" type="fixed">
+    <parent link="Camera-Model-v3"/><child link="front_camera_collision_proxy"/><origin xyz="0 0 0" rpy="0 0 0"/>
+  </joint>
   <!-- SO-101 aggregate links already contain their servo housings. These
        CAD-bounds-derived envelopes therefore cover each complete moving link. -->

Commit message: fix: preserve folded arm clearance with per-part CAD hulls

File: urdf/lekiwi.urdf.xacro (robot description, xacro)
@@ -124,14 +124,4 @@
   <!-- Collision proxies stay attached to their CAD links. Prefer exact
        vendored meshes where enclosing primitives create false collisions. -->
-  <xacro:macro name="collision_capsule_proxy" params="name parent xyz rpy radius cylinder_length">
-    <link name="${name}">
-      <collision><geometry><cylinder radius="${radius}" length="${cylinder_length}"/></geometry></collision>
-      <collision><origin xyz="0 0 ${cylinder_length / 2.0}"/><geometry><sphere radius="${radius}"/></geometry></collision>
-      <collision><origin xyz="0 0 ${-cylinder_length / 2.0}"/><geometry><sphere radius="${radius}"/></geometry></collision>
-    </link>
-    <joint name="${name}_mount" type="fixed">
-      <parent link="${parent}"/><child link="${name}"/><origin xyz="${xyz}" rpy="${rpy}"/>
-    </joint>
-  </xacro:macro>
   <!-- Exact CAD collision meshes avoid the pedestal sphere/upper-arm capsule
        overlapping in poses where the physical parts are separated. -->
@@ -153,7 +143,15 @@
     <parent link="Camera-Model-v3"/><child link="front_camera_collision_proxy"/><origin xyz="0 0 0" rpy="0 0 0"/>
   </joint>
-  <!-- SO-101 aggregate links already contain their servo housings. These
-       CAD-bounds-derived envelopes therefore cover each complete moving link. -->
-  <xacro:collision_capsule_proxy name="shoulder_collision_proxy" parent="so101_shoulder_link" xyz="-0.0192 0.0012 -0.0091" rpy="0 0 0" radius="0.0458" cylinder_length="0.0190"/>
+  <!-- A single enclosing capsule fills the clearance between folded links.
+       Per-part hulls enclose each CAD part's occupied 1 mm cells, preserving
+       those gaps without loading the dense visual meshes into collision checks. -->
+  <link name="shoulder_collision_proxy">
+    <collision><origin xyz="-0.0303992 0.000422241 -0.0417" rpy="1.5708 1.5708 0"/><geometry><mesh filename="package://lekiwi_rmf/urdf/collision/so101_shoulder_link-0.stl"/></geometry></collision>
+    <collision><origin xyz="-0.0675992 -0.000177759 0.0158499" rpy="1.5708 -1.5708 0"/><geometry><mesh filename="package://lekiwi_rmf/urdf/collision/so101_shoulder_link-1.stl"/></geometry></collision>
+    <collision><origin xyz="0.0122008 2.22413e-05 0.0464" rpy="-1.5708 2.35221e-33 0"/><geometry><mesh filename="package://lekiwi_rmf/urdf/collision/so101_shoulder_link-2.stl"/></geometry></collision>
+  </link>
+  <joint name="shoulder_collision_proxy_mount" type="fixed">
+    <parent link="so101_shoulder_link"/><child link="shoulder_collision_proxy"/>
+  </joint>
   <link name="upper_arm_collision_proxy">
     <collision><origin xyz="-0.11257 -0.0155 0.0187" rpy="-3.14159 -5.27356e-16 -1.5708"/><geometry><mesh filename="package://lekiwi_rmf/urdf/meshes/so101/sts3215_03a_v1.stl"/></geometry></collision>
@@ -163,13 +161,18 @@
     <parent link="so101_upper_arm_link"/><child link="upper_arm_collision_proxy"/><origin xyz="0 0 0" rpy="0 0 0"/>
   </joint>
-  <xacro:collision_capsule_proxy name="forearm_collision_proxy" parent="so101_lower_arm_link" xyz="-0.0666 0.0035 0.0202" rpy="0 1.5708 0" radius="0.0411" cylinder_length="0.0749"/>
-  <!-- Native wrist bounds plus 4 mm on each face. The old enclosing sphere
-       extended into the moving jaw even in the reference pose. -->
+  <link name="forearm_collision_proxy">
+    <collision><origin xyz="-0.0648499 -0.032 0.0182" rpy="3.14159 -0 6.67202e-31"/><geometry><mesh filename="package://lekiwi_rmf/urdf/collision/so101_lower_arm_link-0.stl"/></geometry></collision>
+    <collision><origin xyz="-0.0648499 -0.032 0.018" rpy="-3.14159 -2.55351e-15 -1.83387e-30"/><geometry><mesh filename="package://lekiwi_rmf/urdf/collision/so101_lower_arm_link-1.stl"/></geometry></collision>
+    <collision><origin xyz="-0.1224 0.0052 0.0187" rpy="-3.14159 -7.88861e-31 -3.14159"/><geometry><mesh filename="package://lekiwi_rmf/urdf/collision/so101_lower_arm_link-2.stl"/></geometry></collision>
+  </link>
+  <joint name="forearm_collision_proxy_mount" type="fixed">
+    <parent link="so101_lower_arm_link"/><child link="forearm_collision_proxy"/>
+  </joint>
   <link name="wrist_collision_proxy">
-    <collision><geometry><box size="0.04335 0.08584 0.07031"/></geometry></collision>
+    <collision><origin xyz="8.32667e-17 -0.0424 0.0306" rpy="1.5708 1.5708 0"/><geometry><mesh filename="package://lekiwi_rmf/urdf/collision/so101_wrist_link-0.stl"/></geometry></collision>
+    <collision><origin xyz="0 -0.028 0.0181" rpy="-1.5708 -1.5708 0"/><geometry><mesh filename="package://lekiwi_rmf/urdf/collision/so101_wrist_link-1.stl"/></geometry></collision>
   </link>
   <joint name="wrist_collision_proxy_mount" type="fixed">
     <parent link="so101_wrist_link"/><child link="wrist_collision_proxy"/>
-    <origin xyz="-0.00233 -0.026915 0.02215"/>
   </joint>
   <link name="roll_collision_proxy">

Commit message: fix: model folded resting contacts and retain travel stow

File: urdf/lekiwi.urdf.xacro (robot description, xacro)
@@ -147,10 +147,20 @@
        those gaps without loading the dense visual meshes into collision checks. -->
   <link name="shoulder_collision_proxy">
-    <collision><origin xyz="-0.0303992 0.000422241 -0.0417" rpy="1.5708 1.5708 0"/><geometry><mesh filename="package://lekiwi_rmf/urdf/collision/so101_shoulder_link-0.stl"/></geometry></collision>
-    <collision><origin xyz="-0.0675992 -0.000177759 0.0158499" rpy="1.5708 -1.5708 0"/><geometry><mesh filename="package://lekiwi_rmf/urdf/collision/so101_shoulder_link-1.stl"/></geometry></collision>
     <collision><origin xyz="0.0122008 2.22413e-05 0.0464" rpy="-1.5708 2.35221e-33 0"/><geometry><mesh filename="package://lekiwi_rmf/urdf/collision/so101_shoulder_link-2.stl"/></geometry></collision>
   </link>
   <joint name="shoulder_collision_proxy_mount" type="fixed">
     <parent link="so101_shoulder_link"/><child link="shoulder_collision_proxy"/>
+  </joint>
+  <link name="shoulder_motor_collision_proxy">
+    <collision><origin xyz="-0.0303992 0.000422241 -0.0417" rpy="1.5708 1.5708 0"/><geometry><mesh filename="package://lekiwi_rmf/urdf/collision/so101_shoulder_link-0.stl"/></geometry></collision>
+  </link>
+  <joint name="shoulder_motor_collision_proxy_mount" type="fixed">
+    <parent link="so101_shoulder_link"/><child link="shoulder_motor_collision_proxy"/>
+  </joint>
+  <link name="shoulder_holder_collision_proxy">
+    <collision><origin xyz="-0.0675992 -0.000177759 0.0158499" rpy="1.5708 -1.5708 0"/><geometry><mesh filename="package://lekiwi_rmf/urdf/collision/so101_shoulder_link-1.stl"/></geometry></collision>
+  </link>
+  <joint name="shoulder_holder_collision_proxy_mount" type="fixed">
+    <parent link="so101_shoulder_link"/><child link="shoulder_holder_collision_proxy"/>
   </joint>
   <link name="upper_arm_collision_proxy">
@@ -162,10 +172,20 @@
   </joint>
   <link name="forearm_collision_proxy">
-    <collision><origin xyz="-0.0648499 -0.032 0.0182" rpy="3.14159 -0 6.67202e-31"/><geometry><mesh filename="package://lekiwi_rmf/urdf/collision/so101_lower_arm_link-0.stl"/></geometry></collision>
-    <collision><origin xyz="-0.0648499 -0.032 0.018" rpy="-3.14159 -2.55351e-15 -1.83387e-30"/><geometry><mesh filename="package://lekiwi_rmf/urdf/collision/so101_lower_arm_link-1.stl"/></geometry></collision>
     <collision><origin xyz="-0.1224 0.0052 0.0187" rpy="-3.14159 -7.88861e-31 -3.14159"/><geometry><mesh filename="package://lekiwi_rmf/urdf/collision/so101_lower_arm_link-2.stl"/></geometry></collision>
   </link>
   <joint name="forearm_collision_proxy_mount" type="fixed">
     <parent link="so101_lower_arm_link"/><child link="forearm_collision_proxy"/>
+  </joint>
+  <link name="forearm_link_collision_proxy">
+    <collision><origin xyz="-0.0648499 -0.032 0.0182" rpy="3.14159 -0 6.67202e-31"/><geometry><mesh filename="package://lekiwi_rmf/urdf/collision/so101_lower_arm_link-0.stl"/></geometry></collision>
+  </link>
+  <joint name="forearm_link_collision_proxy_mount" type="fixed">
+    <parent link="so101_lower_arm_link"/><child link="forearm_link_collision_proxy"/>
+  </joint>
+  <link name="forearm_holder_collision_proxy">
+    <collision><origin xyz="-0.0648499 -0.032 0.018" rpy="-3.14159 -2.55351e-15 -1.83387e-30"/><geometry><mesh filename="package://lekiwi_rmf/urdf/collision/so101_lower_arm_link-1.stl"/></geometry></collision>
+  </link>
+  <joint name="forearm_holder_collision_proxy_mount" type="fixed">
+    <parent link="so101_lower_arm_link"/><child link="forearm_holder_collision_proxy"/>
   </joint>
   <link name="wrist_collision_proxy">
@@ -178,8 +198,13 @@
   <link name="roll_collision_proxy">
     <collision><origin xyz="0.0077 0.0001 -0.0234" rpy="-1.5708 -5.19179e-17 -1.66533e-16"/><geometry><mesh filename="package://lekiwi_rmf/urdf/meshes/so101/sts3215_03a_v1.stl"/></geometry></collision>
-    <collision><origin xyz="8.32667e-17 -0.000218214 0.000949706" rpy="-3.14159 -5.55112e-17 0"/><geometry><mesh filename="package://lekiwi_rmf/urdf/meshes/so101/wrist_roll_follower_so101_v1.stl"/></geometry></collision>
   </link>
   <joint name="roll_collision_proxy_mount" type="fixed">
     <parent link="so101_gripper_link"/><child link="roll_collision_proxy"/>
+  </joint>
+  <link name="roll_holder_collision_proxy">
+    <collision><origin xyz="8.32667e-17 -0.000218214 0.000949706" rpy="-3.14159 -5.55112e-17 0"/><geometry><mesh filename="package://lekiwi_rmf/urdf/meshes/so101/wrist_roll_follower_so101_v1.stl"/></geometry></collision>
+  </link>
+  <joint name="roll_holder_collision_proxy_mount" type="fixed">
+    <parent link="so101_gripper_link"/><child link="roll_holder_collision_proxy"/>
   </joint>
   <link name="gripper_collision_proxy">

File: urdf/lekiwi_cad.urdf (robot description, URDF)
Before this commit: robot LeKiwi, 39 links, 38 joints
Joints:
- joint arm_shoulder_lift: limit lower=-1.74533 upper=1.82 effort=4 velocity=2 -> lower=-1.825 upper=1.82 effort=4 velocity=2
