Commit message: feat(urdf): vendor the RPi 5 stack and give MoveIt its collision envelope
Vendors robotmindio/LeKiwi a47d47f, which adds the RobotSkin 12x10 through
plate, USB carrier and protection table at the rear right. A box proxy
encloses the stack for self-collision; DEFERRED records the LD06 self-mask
re-measurement the table legs require.

Co-Authored-By: Claude Opus 5.5 (1M context) <noreply@anthropic.com>

File: urdf/lekiwi.urdf.xacro (robot description, xacro)
@@ -156,4 +156,14 @@
     <parent link="ld06_body"/><child link="lidar_collision_proxy"/>
     <origin xyz="0 0 0" rpy="0 0 0"/>
+  </joint>
+  <!-- RPi 5 stack: 12x10 through plate, USB carrier and 30 mm-clearance table.
+       The table encloses both PCBs, so its plate-frame bounds plus 4 mm cover
+       the whole stack (test_collision_model). -->
+  <link name="rpi5_stack_collision_proxy">
+    <collision><geometry><box size="0.128 0.108 0.046"/></geometry></collision>
+  </link>
+  <joint name="rpi5_stack_collision_proxy_mount" type="fixed">
+    <parent link="rpi5_through_plate"/><child link="rpi5_stack_collision_proxy"/>
+    <origin xyz="0 0 0.019" rpy="0 0 0"/>
   </joint>
   <!-- Gazebo-only contact and actuator model.  The CAD wheel meshes and their

File: urdf/lekiwi_cad.urdf (robot description, URDF)
Before this commit: robot LeKiwi, 36 links, 35 joints
Links:
- added link rpi5_table; visual mesh filename=package://lekiwi_rmf/urdf/meshes/rpi5_table.stl scale=0.001 0.001 0.001
- added link rpi5_through_plate; visual mesh filename=package://lekiwi_rmf/urdf/meshes/rpi5_through_plate.stl scale=0.001 0.001 0.001
- added link rpi5_usb_carrier; visual mesh filename=package://lekiwi_rmf/urdf/meshes/rpi5_usb_carrier.stl scale=0.001 0.001 0.001
Joints:
- added joint rpi5_table_joint: type fixed, parent rpi5_through_plate, child rpi5_table, origin xyz=0.0 0.0 0.004 rpy=0 0 0
- added joint rpi5_through_plate_joint: type fixed, parent base_plate_layer2-v3, child rpi5_through_plate, origin xyz=0.125 -0.075 0.007 rpy=0.0 0.0 -1.5707963267948966
- added joint rpi5_usb_carrier_joint: type fixed, parent rpi5_through_plate, child rpi5_usb_carrier, origin xyz=0.0 0.0 0.004 rpy=0 0 0

Commit message: fix(urdf): put the wheels on the floor and the chassis guard on the top deck
base_footprint_to_base_link was 0.093 m, carried over from the old simplified
model; with the vendored CAD the omni-wheel rims reach 40.6 mm below
base_link, so the whole robot (and every sensor frame) was drawn 52 mm above
the floor. Recorded floor-resting arm poses confirm it: they now touch the
floor within 4-17 mm (arm calibration error) instead of hovering 35-48 mm
above it, so MoveIt's exact floor keepout no longer admits plans up to 52 mm
into the real floor.

The D-shaped chassis guard was centred on the lower plate; it is meant to
keep the arm out of the cables above the Raspberry Pi and sensors, so it now
rests on the top plate. The Astra body and lidar proxy are bolted inside
that volume, so their pairs with base_link are exempt like the Pi stack.

Floor-resting e2e poses now assert floor-only contact within the 2 cm
calibration bound, and the floor-reach pose stops where the roll holder
grazes the floor.

Co-Authored-By: Claude Opus 5.5 (1M context) <noreply@anthropic.com>

File: urdf/lekiwi.urdf.xacro (robot description, xacro)
@@ -34,21 +34,24 @@
   <link name="base_footprint"/>
   <link name="base_link">
-    <!-- Keep only the rear of the chassis guard. Its front cut is tangent to
-         the center-facing edge of the arm pedestal; the lower face stays at
-         z=48 mm above the floor, with a 50 mm height. -->
+    <!-- Keep the arm out of the cables above the Raspberry Pi and sensors on
+         the top deck. Only the rear is guarded: the front cut is tangent to the
+         center-facing edge of the arm pedestal. The 50 mm volume rests on the
+         top plate, whose upper face is 57 mm above base_link. -->
     <collision>
-      <origin xyz="0 0 -0.020"/>
+      <origin xyz="0 0 0.082"/>
       <geometry><mesh filename="package://lekiwi_rmf/urdf/chassis_guard.stl"/></geometry>
     </collision>
     <!-- Show the exact restricted volume in the default RViz RobotModel. -->
     <visual>
-      <origin xyz="0 0 -0.020"/>
+      <origin xyz="0 0 0.082"/>
       <geometry><mesh filename="package://lekiwi_rmf/urdf/chassis_guard.stl"/></geometry>
       <material name="chassis_guard"><color rgba="1 0.2 0.1 0.5"/></material>
     </visual>
   </link>
+  <!-- The CAD's omni-wheel rims reach 40.6 mm below the lower plate's top
+       face (base_link), so this places the wheel-contact plane on the floor. -->
   <joint name="base_footprint_to_base_link" type="fixed">
     <parent link="base_footprint"/><child link="base_link"/>
-    <origin xyz="0 0 0.093" rpy="0 0 0"/>
+    <origin xyz="0 0 0.0406" rpy="0 0 0"/>
   </joint>
   <!-- The wheel-contact plane is the floor. Keep modeled parts above it while
